File: pcb/diplomen_proekt.kicad_pcb (KiCad board)
At the start: 2 copper layers, 80.1 x 96 mm, 24 parts, among them SW1 SW_Push, U1 DA56-11SURKWA, U2 ESP32-S3, U3 HC-SR04, U4 ACTIVE_BUZZER, U5 TP4056, U6 MCP1826S

Commit message: Added capacitors
Parts:
- added C1: 1uF, Capacitor_THT:CP_Radial_D5.0mm_P2.50mm, F.Cu at (173.4, 57.9)
- added C2: 1uF, Capacitor_THT:CP_Radial_D5.0mm_P2.50mm, F.Cu at (162.0, 51.0)
- added C3: 0.1uF, Capacitor_THT:CP_Radial_D5.0mm_P2.50mm, F.Cu at (153.5, 116.4)
- moved U6 64.8 mm to (158.2, 51.0)
- turned BT2 to -90 degrees
Connections:
- SW1 pad 2: GND -> Net-(C3-Pad1)
- U6 pad 1: BAT -> Net-(U6-VI)
- U6 pad 3: +3.3V -> Net-(U6-VO)
Routing:
- net +3.3V: track 162.9 -> 117.7 mm, vias 4 -> 2
- net BAT: track 135.7 -> 156.4 mm, vias 3 -> 0
- net Net-(U6-VI): track 0.00 -> 16.5 mm
- net Net-(C3-Pad1): track 0.00 -> 10.6 mm
- net Net-(U6-VO): track 0.00 -> 4.77 mm
- net GND: track 0.00 -> 2.59 mm, vias 0 -> 1

Commit message: Added pcb images
Routing:
- net +3.3V: track 117.7 -> 118.5 mm
Changed lines of the file:
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@@
 		(tags "CP Radial series Radial pin pitch 2.50mm  diameter 5mm Electrolytic Capacitor")
 		(property "Reference" "C3"
-			(at 1.25 -3.75 360)
+			(at 1.25 -3.75 0)
 			(layer "F.SilkS")
 			(effects
@@
 		)
 		(property "Value" "0.1uF"
-			(at 1.25 3.75 360)
+			(at 1.25 3.75 0)
 			(layer "F.Fab")
 			(effects
@@
 		)
 		(fp_text user "${REFERENCE}"
-			(at 1.25 0 360)
+			(at 1.25 0 0)
 			(layer "F.Fab")
 			(effects
@@
 		)
 		(fp_text user "${REFERENCE}"
-			(at -0.05 -0.83 0)
+			(at -0.05 1.8 0)
 			(unlocked yes)
 			(layer "F.Fab")
@@
 		(tags "Through hole angled socket strip THT 1x04 2.54mm single row")
 		(property "Reference" "U3"
-			(at -4.38 -2.77 90)
+			(at -5.8 3.75 180)
 			(layer "F.SilkS")
 			(effects
@@
 		(tags "Display")
 		(property "Reference" "U1"
-			(at 0 0 0)
+			(at 6.22 -0.8 0)
 			(layer "F.SilkS")
 			(effects
@@
 		(attr through_hole)
 		(fp_line
-			(start -2.03 -2.465)
-			(end -2.03 0)
+			(start -2.03 22.785)
+			(end -2.03 -2.465)
 			(stroke
 				(width 0.2)
-				(type solid)
+				(type default)
 			)
 			(layer "F.SilkS")
@@
 		)
 		(fp_line
+			(start 17.27 -2.465)
+			(end 17.27 22.785)
+			(stroke
+				(width 0.2)
+				(type default)
+			)
+			(layer "F.SilkS")
+		)
+		(fp_line
 			(start -2.28 -2.715)
 			(end 17.52 -2.715)
@@
 		)
 		(fp_text user "${REFERENCE}"
-			(at 0 0 0)
+			(at 6.22 -0.8 0)
 			(layer "F.Fab")
 			(effects
@@
 		(at 167.1 98.39 -90)
 		(property "Reference" "BT2"
-			(at -34.925 -11.43 90)
+			(at 0 0 90)
 			(layer "F.SilkS")
 			(effects
@@
 	)
 	(segment
-		(start 164.514888 51)
-		(end 164.514888 53.6)
-		(width 1)
-		(layer "F.Cu")
-		(net 2)
-	)
-	(segment
 		(start 125.71 75.2)
 		(end 122.2 78.71)
@@
 	)
 	(segment
-		(start 164.514888 55.985112)
-		(end 164.5 56)
-		(width 1)
-		(layer "F.Cu")
-		(net 2)
-	)
-	(segment
 		(start 133 59.08)
 		(end 134.92 57.16)
@@
 	)
 	(segment
-		(start 156.3 64.2)
-		(end 156.3 75.2)
-		(width 1)
-		(layer "F.Cu")
-		(net 2)
-	)
-	(segment
 		(start 125.71 67.902373)
 		(end 133 60.612373)
@@
 	)
 	(segment
-		(start 164.5 56)
-		(end 156.3 64.2)
+		(start 156.3 75.2)
+		(end 156.3 63.93)
 		(width 1)
 		(layer "F.Cu")
@@
 	)
 	(segment
-		(start 166.63 53.6)
-		(end 168.53 51.7)
+		(start 149 75.2)
+		(end 125.71 75.2)
 		(width 1)
 		(layer "F.Cu")
@@
 	)
 	(segment
-		(start 149 75.2)
-		(end 125.71 75.2)
+		(start 164.715 55.515)
+		(end 168.53 51.7)
 		(width 1)
 		(layer "F.Cu")
@@
 	)
 	(segment
-		(start 125.71 75.2)
-		(end 125.71 67.902373)
+		(start 164.715 55.515)
+		(end 164.514888 55.314888)
 		(width 1)
 		(layer "F.Cu")
@@
 	)
 	(segment
-		(start 164.514888 53.6)
-		(end 164.514888 55.985112)
+		(start 164.514888 55.314888)
+		(end 164.514888 51)
+		(width 1)
+		(layer "F.Cu")
+		(net 2)
+	)
+	(segment
+		(start 125.71 75.2)
+		(end 125.71 67.902373)
 		(width 1)
 		(layer "F.Cu")
@@
 	)
 	(segment
-		(start 164.514888 53.6)
-		(end 166.63 53.6)
+		(start 156.3 63.93)
+		(end 164.715 55.515)
 		(width 1)
 		(layer "F.Cu")
@@
 		(min_thickness 0.25)
 		(filled_areas_thickness no)
-		(fill
+		(fill yes
 			(thermal_gap 0.5)
 			(thermal_bridge_width 0.5)
